Commit message: Replace primitive geometry with SolidWorks STL mesh model; fix Z-up orientation and center robot at origin

File: src/auto_car_description/urdf/auto_car.urdf (robot description, URDF)
Before this commit: robot auto_car, 9 links, 8 joints
Links:
- removed link cover_lower
- removed link cover_upper
- removed link wheel_front_left
- removed link wheel_front_right
- removed link wheel_rear_left
- removed link wheel_rear_right
- added link back_left_wheel_link, mass 0.0536934866827212; collision mesh filename=package://auto_car_description/meshes/back_left_wheel_link.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; visual mesh filename=package://auto_car_description/meshes/back_left_wheel_link.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
- added link back_right_wheel_link, mass 0.0536235654025979; collision mesh filename=package://auto_car_description/meshes/back_right_wheel_link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; visual mesh filename=package://auto_car_description/meshes/back_right_wheel_link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
- added link chassis_link, mass 0.587421422264195; collision mesh filename=package://auto_car_description/meshes/chassis_link.STL; visual mesh filename=package://auto_car_description/meshes/chassis_link.STL
- added link front_left_wheel_link, mass 0.0536235654026291; collision mesh filename=package://auto_car_description/meshes/front_left_wheel_link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; visual mesh filename=package://auto_car_description/meshes/front_left_wheel_link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
- added link front_right_wheel_link, mass 0.0536934866822392; collision mesh filename=package://auto_car_description/meshes/front_right_wheel_lin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; visual mesh filename=package://auto_car_description/meshes/front_right_wheel_lin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
- link base_link: mass 2.0 -> None; geometry 
- link lidar_link: mass 0.17 -> 0.102513123166222; geometry collision mesh filename=package://auto_car_description/meshes/lidar_link.STL; visual mesh filename=package://auto_car_description/meshes/lidar_link.STL
Joints:
- removed joint joint_cover_lower
- removed joint joint_cover_upper
- removed joint joint_front_left
- removed joint joint_front_right
- removed joint joint_lidar
- removed joint joint_rear_left
- removed joint joint_rear_right
- added joint back_left_wheel_joint: type continuous, parent chassis_link, child back_left_wheel_link, origin xyz=0.77108 -1.432 0.91691 rpy=0 0 3.1416, axis 0 -1 0
- added joint back_right_wheel_joint: type continuous, parent chassis_link, child back_right_wheel_link, origin xyz=0.77108 -1.2445 0.91691 rpy=0 0 3.1416, axis 0 -1 0
- added joint chassis_joint: type fixed, parent base_link, child chassis_link, origin xyz=-0.6986 1.338 -0.88691
- added joint front_left_wheel_joint: type continuous, parent chassis_link, child front_left_wheel_link, origin xyz=0.62608 -1.432 0.91691 rpy=0 0 3.1416, axis 0 1 0
- added joint front_right_wheel_joint: type continuous, parent chassis_link, child front_right_wheel_link, origin xyz=0.62608 -1.2445 0.91691 rpy=0 0 3.1416, axis 0 1 0
- added joint lidar_joint: type fixed, parent chassis_link, child lidar_link, origin xyz=0.74291 -1.3383 1.0394 rpy=0 0 3.1416, axis 0 0 0
- joint base_footprint_joint: origin xyz=0 0 0.0165 rpy=0 0 0 -> xyz=0 0 0 rpy=0 0 0

Commit message: Replace primitive geometry with SolidWorks STL meshes; fix orientation, centering, collision shapes, and inertial origin; add Gazebo mesh resource path

File: src/auto_car_description/urdf/auto_car.urdf (robot description, URDF)
Before this commit: robot assembly_for_urdf, 8 links, 7 joints
Links:
- link back_left_wheel_link: geometry collision cylinder length=0.030 radius=0.030; visual mesh filename=package://auto_car_description/meshes/back_left_wheel_link.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
- link back_right_wheel_link: geometry collision cylinder length=0.030 radius=0.030; visual mesh filename=package://auto_car_description/meshes/back_right_wheel_link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
- link chassis_link: geometry collision box size=0.22713 0.121 0.033; visual mesh filename=package://auto_car_description/meshes/chassis_link.STL
- link front_left_wheel_link: geometry collision cylinder length=0.030 radius=0.030; visual mesh filename=package://auto_car_description/meshes/front_left_wheel_link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
- link front_right_wheel_link: geometry collision cylinder length=0.030 radius=0.030; visual mesh filename=package://auto_car_description/meshes/front_right_wheel_lin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
